File: kicad_7_files/highQ.kicad_pcb (KiCad board)
At the start: 4 copper layers, 36 parts, among them U1 INA128, U2 OPA188xxD, U3 LT3092xST, U4 REF3025

Commit message: Updated Readme and Rg Value
Parts:
- R5: value 2.5K -> 1.6K
Connections:
- net +12V renamed Net-(C3-Pad2)
- C17 pad 2: +5V -> Net-(U4-IN)
- C19 pad 2: +5V -> Net-(U2-V+)
- C21 pad 2: +5V -> Net-(U2-V+)
- C24 pad 2: +5V -> Net-(U4-IN)
- C5 pad 2: +5V -> Net-(U1-V+)
- C7 pad 2: +5V -> Net-(U1-V+)
- U1 pad 7: +5V -> Net-(U1-V+)
- U2 pad 7: +5V -> Net-(U2-V+)
- U4 pad 1: +5V -> Net-(U4-IN)
Routing:
- net Net-(U4-IN): track 0.00 -> 6.11 mm
- net +5V: track 6.11 -> 0.00 mm
Changed lines of the file:
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@@
   (net 12 "Net-(U2-+)")
   (net 13 "Output")
-  (net 14 "+12V")
+  (net 14 "Net-(C3-Pad2)")
   (net 15 "Net-(C12-Pad2)")
   (net 16 "Net-(C22-Pad1)")
@@
   (net 20 "unconnected-(U2-NC-Pad5)")
   (net 21 "unconnected-(U2-NC-Pad8)")
-  (net 22 "+5V")
+  (net 22 "Net-(U1-V+)")
+  (net 23 "Net-(U4-IN)")
+  (net 24 "Net-(U2-V+)")
   (footprint "Capacitor_SMD:C_0603_1608Metric" (layer "F.Cu")
     (at 104.058491 75.139701 -90)
@@
       (net 6 "GND") (pintype "passive"))
     (pad "2" smd roundrect (at 0.775 0 270) (size 0.9 0.95) (layers "F.Cu" "F.Paste" "F.Mask") (roundrect_rratio 0.25)
-      (net 22 "+5V") (pintype "passive"))
+      (net 23 "Net-(U4-IN)") (pintype "passive"))
     (model "${KICAD6_3DMODEL_DIR}/Capacitor_SMD.3dshapes/C_0603_1608Metric.wrl"
       (offset (xyz 0 0 0))
@@
         (effects (font (size 1 1) (thickness 0.15)))
     )
-    (fp_text value "2.5K" (at 0 1.43 90) (layer "F.Fab") hide
+    (fp_text value "1.6K" (at 0 1.43 90) (layer "F.Fab") hide
         (effects (font (size 1 1) (thickness 0.15)))
     )
@@
       (net 18 "Net-(R10-Pad2)") (pintype "output"))
     (pad "7" smd roundrect (at 2.475 -0.635 270) (size 1.95 0.6) (layers "F.Cu" "F.Paste" "F.Mask") (roundrect_rratio 0.25)
-      (net 22 "+5V") (pinfunction "V+") (pintype "power_in"))
+      (net 22 "Net-(U1-V+)") (pinfunction "V+") (pintype "power_in"))
     (pad "8" smd roundrect (at 2.475 -1.905 270) (size 1.95 0.6) (layers "F.Cu" "F.Paste" "F.Mask") (roundrect_rratio 0.25)
       (net 11 "Net-(R5-Pad2)") (pinfunction "Rg") (pintype "passive"))
@@
       (net 6 "GND") (pintype "passive"))
     (pad "2" smd roundrect (at 0.95 0 90) (size 1 1.45) (layers "F.Cu" "F.Paste" "F.Mask") (roundrect_rratio 0.25)
-      (net 14 "+12V") (pintype "passive"))
+      (net 14 "Net-(C3-Pad2)") (pintype "passive"))
     (model "${KICAD6_3DMODEL_DIR}/Capacitor_SMD.3dshapes/C_0805_2012Metric.wrl"
       (offset (xyz 0 0 0))
@@
       (net 13 "Output") (pintype "output"))
     (pad "7" smd roundrect (at 2.475 -0.635 180) (size 1.95 0.6) (layers "F.Cu" "F.Paste" "F.Mask") (roundrect_rratio 0.25)
-      (net 22 "+5V") (pinfunction "V+") (pintype "power_in"))
+      (net 24 "Net-(U2-V+)") (pinfunction "V+") (pintype "power_in"))
     (pad "8" smd roundrect (at 2.475 -1.905 180) (size 1.95 0.6) (layers "F.Cu" "F.Paste" "F.Mask") (roundrect_rratio 0.25)
       (net 21 "unconnected-(U2-NC-Pad8)") (pinfunction "NC") (pintype "no_connect"))
@@
       (net 6 "GND") (pintype "passive"))
     (pad "2" smd roundrect (at 0.775 0 90) (size 0.9 0.95) (layers "F.Cu" "F.Paste" "F.Mask") (roundrect_rratio 0.25)
-      (net 14 "+12V") (pintype "passive"))
+      (net 14 "Net-(C3-Pad2)") (pintype "passive"))
     (model "${KICAD6_3DMODEL_DIR}/Capacitor_SMD.3dshapes/C_0603_1608Metric.wrl"
       (offset (xyz 0 0 0))
@@
       (net 6 "GND") (pintype "passive"))
     (pad "2" smd roundrect (at 0.95 0) (size 1 1.45) (layers "F.Cu" "F.Paste" "F.Mask") (roundrect_rratio 0.25)
-      (net 22 "+5V") (pintype "passive"))
+      (net 22 "Net-(U1-V+)") (pintype "passive"))
     (model "${KICAD6_3DMODEL_DIR}/Capacitor_SMD.3dshapes/C_0805_2012Metric.wrl"
       (offset (xyz 0 0 0))
@@
       (net 6 "GND") (pintype "passive"))
     (pad "2" smd roundrect (at 0.95 0 270) (size 1 1.45) (layers "F.Cu" "F.Paste" "F.Mask") (roundrect_rratio 0.25)
-      (net 22 "+5V") (pintype "passive"))
+      (net 23 "Net-(U4-IN)") (pintype "passive"))
     (model "${KICAD6_3DMODEL_DIR}/Capacitor_SMD.3dshapes/C_0805_2012Metric.wrl"
       (offset (xyz 0 0 0))
@@
       (stroke (width 0.1) (type solid)) (layer "F.Fab"))
     (pad "1" smd roundrect (at -0.9375 -0.95 90) (size 1.475 0.6) (layers "F.Cu" "F.Paste" "F.Mask") (roundrect_rratio 0.25)
-      (net 22 "+5V") (pinfunction "IN") (pintype "power_in"))
+      (net 23 "Net-(U4-IN)") (pinfunction "IN") (pintype "power_in"))
     (pad "2" smd roundrect (at -0.9375 0.95 90) (size 1.475 0.6) (layers "F.Cu" "F.Paste" "F.Mask") (roundrect_rratio 0.25)
       (net 9 "Net-(U1-Ref)") (pinfunction "OUT") (pintype "power_out"))
@@
       (net 6 "GND") (pintype "passive"))
     (pad "2" smd roundrect (at 0.775 0) (size 0.9 0.95) (layers "F.Cu" "F.Paste" "F.Mask") (roundrect_rratio 0.25)
-      (net 22 "+5V") (pintype "passive"))
+      (net 24 "Net-(U2-V+)") (pintype "passive"))
     (model "${KICAD6_3DMODEL_DIR}/Capacitor_SMD.3dshapes/C_0603_1608Metric.wrl"
       (offset (xyz 0 0 0))
@@
       (net 17 "Net-(R2-Pad2)") (pintype "passive"))
     (pad "3" smd rect (at -3.15 2.3) (size 2 1.5) (layers "F.Cu" "F.Paste" "F.Mask")
-      (net 14 "+12V") (pintype "passive"))
+      (net 14 "Net-(C3-Pad2)") (pintype "passive"))
     (model "${KICAD6_3DMODEL_DIR}/Package_TO_SOT_SMD.3dshapes/SOT-223.wrl"
       (offset (xyz 0 0 0))
@@
       (net 6 "GND") (pintype "passive"))
     (pad "2" smd roundrect (at 0.95 0) (size 1 1.45) (layers "F.Cu" "F.Paste" "F.Mask") (roundrect_rratio 0.25)
-      (net 22 "+5V") (pintype "passive"))
+      (net 24 "Net-(U2-V+)") (pintype "passive"))
     (model "${KICAD6_3DMODEL_DIR}/Capacitor_SMD.3dshapes/C_0805_2012Metric.wrl"
       (offset (xyz 0 0 0))
@@
       (net 6 "GND") (pintype "passive"))
     (pad "2" smd roundrect (at 0.775 0) (size 0.9 0.95) (layers "F.Cu" "F.Paste" "F.Mask") (roundrect_rratio 0.25)
-      (net 22 "+5V") (pintype "passive"))
+      (net 22 "Net-(U1-V+)") (pintype "passive"))
     (model "${KICAD6_3DMODEL_DIR}/Capacitor_SMD.3dshapes/C_0603_1608Metric.wrl"
       (offset (xyz 0 0 0))
@@
   (segment (start 149.808493 89.088855) (end 151.601145 89.088855) (width 0.254) (layer "F.Cu") (net 17))
   (segment (start 151.601145 89.088855) (end 151.79 88.9) (width 0.762) (layer "F.Cu") (net 17))
-  (segment (start 107.037966 76.108488) (end 110.084869 76.108488) (width 0.254) (layer "F.Cu") (net 22))
-  (segment (start 104.058491 75.914701) (end 106.844179 75.914701) (width 0.254) (layer "F.Cu") (net 22))
-  (segment (start 106.844179 75.914701) (end 107.037966 76.108488) (width 0.254) (layer "F.Cu") (net 22))
-  (segment (start 110.084869 76.108488) (end 110.089499 76.103858) (width 0.254) (layer "F.Cu") (net 22))
+  (segment (start 107.037966 76.108488) (end 110.084869 76.108488) (width 0.254) (layer "F.Cu") (net 23))
+  (segment (start 104.058491 75.914701) (end 106.844179 75.914701) (width 0.254) (layer "F.Cu") (net 23))
+  (segment (start 106.844179 75.914701) (end 107.037966 76.108488) (width 0.254) (layer "F.Cu") (net 23))
+  (segment (start 110.084869 76.108488) (end 110.089499 76.103858) (width 0.254) (layer "F.Cu") (net 23))
 )
