File: kicad_7_files/highQ.kicad_sch (KiCad schematic)
At the start: 40 parts, among them U1 INA128, U2 OPA188xxD, U3 LT3092xST, U4 REF3025

Commit message: Updated Readme and Rg Value
Parts:
- R5: value 1.6K -> 2.5K
Changed lines of the file:
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@@
       (effects (font (size 1.27 1.27)))
     )
-    (property "Value" "1.6K" (at 127 85.09 90)
+    (property "Value" "2.5K" (at 127 85.09 90)
       (effects (font (size 1.27 1.27)))
     )
